File: llavero_rfid_hard.kicad_sch (KiCad schematic)
At the start: 11 parts, among them Q1 BC549, SW1 SW_Push, SW2 SW_Push, SW3 SW_Push, SW4 SW_Push, U1 ATtiny85-20P

Commit message: actualizo sch y mejora de version
Parts:
- C1: value 100nF -> 8nF
- L1: value L -> 208uH
- Q1: value BC549 -> 2N3904
- R1: value 10K -> 1K
Changed lines of the file:
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@@
 			)
 		)
-		(property "Value" "BC549"
+		(property "Value" "2N3904"
 			(at 163.83 72.3899 0)
 			(show_name no)
@@
 			)
 		)
-		(property "Value" "10K"
+		(property "Value" "1K"
 			(at 146.05 67.31 90)
 			(show_name no)
@@
 			)
 		)
-		(property "Value" "L"
+		(property "Value" "208uH"
 			(at 191.77 72.3899 0)
 			(show_name no)
@@
 			)
 		)
-		(property "Value" "100nF"
+		(property "Value" "8nF"
 			(at 180.34 72.3899 0)
 			(show_name no)
